File: PWR_MOD.kicad_pcb (KiCad board)
At the start: 4 copper layers, 111.1 x 91.3 mm, 212 parts, among them J1 Barrel_Jack, J11 Conn_01x03, J2 Conn_ARM_JTAG_SWD_20, J3 Conn_01x03, J4 Conn_01x04_Pin, J5 Conn_Coaxial, J6 Conn_01x04_Pin, J7 USB_C_Receptacle_USB2.0_16P, Q1 IRF7341PBF, Q2 SS8050, Q3 SS8050, U1 AD8606ARZ, U10 ADS1232IPW, U11 REF195, U12 ESP32-WROOM-32, U13 CH340C, U14 MCP3551-EMS, U16 TPS60400DBV, U17 CA3140, U18 TL081, U2 LM317_SOT-223, U3 LM2576S-ADJ, U4 STM32F407VETx, U5 24LC256, U6 ADuM1401xRW, U7 LP2985-3.3, U8 REF195, U9 L7809, Y1 8 MHz, Y2 32k

Commit message: redaction_10
Parts:
- moved C27 0.33 mm to (176.3, 110.7)
- moved C26 0.30 mm to (176.1, 113.0)
Changed lines of the file:
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@@
 	(footprint "Capacitor_SMD:C_0805_2012Metric_Pad1.18x1.45mm_HandSolder"
 		(layer "F.Cu")
-		(at 176.0125 110.5 180)
+		(at 176.272 110.7 180)
 		(descr "Capacitor SMD 0805 (2012 Metric), square (rectangular) end terminal, IPC-7351 nominal with elongated pad for handsoldering. (Body size source: IPC-SM-782 page 76, https://www.pcb-3d.com/wordpress/wp-content/uploads/ipc-sm-782a_amendment_1_and_2.pdf, https://docs.google.com/spreadsheets/d/1BsfQQcO9C6DZCsRaXUlFlo91Tg2WpOkGARC1WS5S8t0/edit?usp=sharing)")
 		(tags "capacitor handsolder")
 		(property "Reference" "C27"
-			(at 3.1125 0 0)
+			(at 0 2.032 0)
 			(layer "F.SilkS")
 			(effects
@@
 		(sheetname "/Rx & Tx/")
 		(sheetfile "без_имени.kicad_sch")
-		(units
-			(unit
-				(name "A")
-				(pins "1" "2")
-			)
-		)
 		(attr smd)
 		(duplicate_pad_numbers_are_jumpers no)
-		(fp_line
-			(start -0.261252 0.735)
-			(end 0.261252 0.735)
-			(stroke
-				(width 0.12)
-				(type solid)
-			)
-			(layer "F.SilkS")
-		)
-		(fp_line
-			(start -0.261252 -0.735)
-			(end 0.261252 -0.735)
-			(stroke
-				(width 0.12)
-				(type solid)
-			)
-			(layer "F.SilkS")
-		)
-		(fp_rect
-			(start -1.88 -0.98)
-			(end 1.88 0.98)
-			(stroke
-				(width 0.05)
-				(type solid)
-			)
-			(fill no)
-			(layer "F.CrtYd")
-		)
-		(fp_rect
-			(start -1 -0.625)
-			(end 1 0.625)
-			(stroke
-				(width 0.1)
-				(type solid)
-			)
-			(fill no)
-			(layer "F.Fab")
-		)
 		(pad "1" smd roundrect
-			(at -1.0375 0 180)
-			(size 1.175 1.45)
+			(at -1.778 0 180)
+			(size 2 2)
 			(layers "F.Cu" "F.Mask" "F.Paste")
 			(roundrect_rratio 0.212766)
@@
 		)
 		(pad "2" smd roundrect
-			(at 1.0375 0 180)
-			(size 1.175 1.45)
+			(at 1.778 0 180)
+			(size 2 2)
 			(layers "F.Cu" "F.Mask" "F.Paste")
 			(roundrect_rratio 0.212766)
@@
 	(footprint "Capacitor_SMD:C_0805_2012Metric_Pad1.18x1.45mm_HandSolder"
 		(layer "F.Cu")
-		(at 176.0125 112.7 180)
+		(at 176.05 113 180)
 		(descr "Capacitor SMD 0805 (2012 Metric), square (rectangular) end terminal, IPC-7351 nominal with elongated pad for handsoldering. (Body size source: IPC-SM-782 page 76, https://www.pcb-3d.com/wordpress/wp-content/uploads/ipc-sm-782a_amendment_1_and_2.pdf, https://docs.google.com/spreadsheets/d/1BsfQQcO9C6DZCsRaXUlFlo91Tg2WpOkGARC1WS5S8t0/edit?usp=sharing)")
 		(tags "capacitor handsolder")
@@
 	)
 	(segment
-		(start 177.05 112.7)
-		(end 177.05 110.5)
+		(start 181.0875 113.6625)
+		(end 181.545 113.205)
 		(width 0.2)
 		(layer "F.Cu")
@@
 	)
 	(segment
-		(start 181.0875 113.6625)
-		(end 181.545 113.205)
+		(start 178.05 110.5)
+		(end 178.45 110.5)
+		(width 0.2)
+		(layer "F.Cu")
+		(net "+3.3V1")
+	)
+	(segment
+		(start 178.05 110.1)
+		(end 178.05 108.9)
 		(width 0.2)
 		(layer "F.Cu")
@@
 	)
 	(segment
+		(start 178.45 110.5)
+		(end 178.05 110.1)
+		(width 0.2)
+		(layer "F.Cu")
+		(net "+3.3V1")
+	)
+	(segment
+		(start 177.05 112.7)
+		(end 178.05 111.7)
+		(width 0.2)
+		(layer "F.Cu")
+		(net "+3.3V1")
+	)
+	(segment
 		(start 173.545 125.805)
 		(end 173.65 125.7)
@@
 	)
 	(segment
+		(start 178.05 108.9)
+		(end 178.85 108.1)
+		(width 0.2)
+		(layer "F.Cu")
+		(net "+3.3V1")
+	)
+	(segment
 		(start 177.05 112.7)
 		(end 178.45 112.7)
@@
 	)
 	(segment
-		(start 178.45 110.5)
-		(end 177.05 110.5)
+		(start 178.05 111.7)
+		(end 178.05 110.5)
 		(width 0.2)
 		(layer "F.Cu")
@@
 		(width 0.2)
 		(layer "F.Cu")
-		(net "+3.3V1")
-	)
-	(segment
-		(start 178.85 110.1)
-		(end 178.45 110.5)
-		(width 0.2)
-		(layer "F.Cu")
-		(net "+3.3V1")
-	)
-	(segment
-		(start 178.85 108.1)
-		(end 178.85 110.1)
-		(width 0.2)
-		(layer "F.Cu")

Commit message: redaction_11
Parts:
- removed R38, R39: 1k, Resistor_SMD:R_0805_2012Metric_Pad1.20x1.40mm_HandSolder
- added C31: 0.1 uF, Capacitor_SMD:C_0805_2012Metric_Pad1.18x1.45mm_HandSolder, F.Cu at (139.8, 146.5)
- added R106: 100, Resistor_SMD:R_0805_2012Metric_Pad1.20x1.40mm_HandSolder, F.Cu at (157.8, 152.8)
- added R107: 1k, Resistor_SMD:R_0805_2012Metric_Pad1.20x1.40mm_HandSolder, F.Cu at (157.9, 148.8)
- added R108: 1k, Resistor_SMD:R_0805_2012Metric_Pad1.20x1.40mm_HandSolder, F.Cu at (157.9, 150.8)
- added R109: 1k, Resistor_SMD:R_0805_2012Metric_Pad1.20x1.40mm_HandSolder, F.Cu at (133.0, 146.5)
- added R40: 1k, Resistor_SMD:R_0805_2012Metric_Pad1.20x1.40mm_HandSolder, F.Cu at (137.8, 149.4)
- added R69: 1k, Resistor_SMD:R_0805_2012Metric_Pad1.20x1.40mm_HandSolder, F.Cu at (157.9, 146.8)
- added R70: 1k, Resistor_SMD:R_0805_2012Metric_Pad1.20x1.40mm_HandSolder, F.Cu at (137.8, 151.3)
- added R71: 1k, Resistor_SMD:R_0805_2012Metric_Pad1.20x1.40mm_HandSolder, F.Cu at (137.8, 153.2)
- added R72: 100, Resistor_SMD:R_0805_2012Metric_Pad1.20x1.40mm_HandSolder, F.Cu at (136.7, 147.5)
- added U19: ADuM1401xRW, Package_SO:SOIC-16W_7.5x10.3mm_P1.27mm, F.Cu at (148.1, 149.7)
Connections:
- U10 pad 23: SCK_1 -> SCLK_ADS1232
- U10 pad 24: SDO_1 -> DOUT_ADS1232
- U4 pad 78: unconnected-(U4-PC10-Pad78) -> SCK_STM32_AD1232
- U4 pad 79: unconnected-(U4-PC11-Pad79) -> MISO_AD1232
- U4 pad 80: unconnected-(U4-PC12-Pad80) -> MOSI_AD1232
- U6 pad 12: Net-(U6-VOC) -> unconnected-(U6-VOC-Pad12)
- U6 pad 5: Net-(U6-VIC) -> GND_0
Routing:
- net MISO_AD1232: track 0.00 -> 76.6 mm, vias 0 -> 3
- net SCK_STM32_AD1232: track 0.00 -> 73.5 mm, vias 0 -> 3
- net MOSI_AD1232: track 0.00 -> 66.2 mm, vias 0 -> 4
- net CS_ADS1232: track 52.2 -> 86.6 mm, vias 4 -> 5
- net DOUT_ADS1232: track 0.00 -> 29.0 mm, vias 0 -> 2
- net SCLK_ADS1232: track 0.00 -> 25.1 mm, vias 0 -> 2
- net Net-(U19-VDD1): track 0.00 -> 21.2 mm, vias 0 -> 2
- net Net-(U19-VDD2): track 0.00 -> 17.8 mm, vias 0 -> 1
- net SCK_1: track 27.8 -> 10.2 mm, vias 2 -> 1
- net CS_1232: track 11.9 -> 25.8 mm
- net SDO_1: track 20.7 -> 9.82 mm, vias 3 -> 2
- net GND_0: track 220.6 -> 229.3 mm, vias 128 -> 132
- net Net-(U19-VIB): track 0.00 -> 6.37 mm
- net Net-(U19-VOD): track 0.00 -> 5.69 mm
- net Net-(U19-VIA): track 0.00 -> 5.41 mm
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Other:
- board size 111.1 x 91.3 mm -> 111.1 x 101.7 mm
