File: без_имени.kicad_sch (KiCad schematic)
At the start: 70 parts, among them Q1 IRF7341PBF, U1 AD8606ARZ, U10 ADS1232IPW, U11 REF195, U14 MCP3551-EMS, U16 TPS60400DBV, U6 ADuM1401xRW, U7 LP2985-3.3, U8 REF195, U9 L7809

Commit message: redaction_11
Parts:
- removed R38, R39: 1k, Resistor_SMD:R_0805_2012Metric_Pad1.20x1.40mm_HandSolder, symbol Device:R
Connections:
- net GND_0: now also U6.5 (VIC)
- net SCK_1: no longer U10.23 (SCLK)
- net SDO_1: no longer U10.24 (~{DRDY}/DOUT)
- new net DOUT_ADS1232: U10.24 (~{DRDY}/DOUT)
- new net SCLK_ADS1232: U10.23 (SCLK)
- no-connect marks 4 -> 5
